Commit message: Added example controller.

File: Simscape/URDF/urdf/SMART NS 12-1,85_ARTICOLATO.SLDASM.urdf (robot description, URDF)
Before this commit: robot SMART NS 12-1,85_ARTICOLATO.SLDASM, 7 links, 6 joints
Links:
- link Link1: mass 45.9345551191719 -> 45.9345542594997
- link Link2: mass 7.5113 -> 7.51128820326683
- link Link3: mass 21.7051356161458 -> 21.7051384673217
- link Link4: mass 5.72544134618086 -> 5.72544149128189
- link Link5: mass 0.559213525407613 -> 0.559213536738551
- link LinkBase: mass 49.7889558189811 -> 49.7889558845622
- link LinkEE: mass 0.091959 -> 0.0919593711752515
Joints:
- joint Ax1: origin xyz=-0.51441 -1.058 0 rpy=1.5708 0 0.1238 -> xyz=0 0 0.251 rpy=1.5708 0 0
- joint Ax2: origin xyz=-0.3 -0.092964 -0.067936 rpy=0 0 -7.8035E-05 -> xyz=-0.3 0.349 -0.101 rpy=0 0 -7.8035E-05
- joint Ax4: origin xyz=-0.24805 0.185 0.067936 rpy=0 0 0 -> xyz=-0.238 0.185 0.101 rpy=0 0 0
- joint Ax5: origin xyz=-0.58195 0 0 rpy=0 0 0.016772 -> xyz=-0.592 0 0 rpy=0 0 0.016135
- joint Ax6: origin xyz=-0.093054 0 0 rpy=-1.5528 0 0 -> xyz=-0.092478 0 0 rpy=-1.5434 0 0

Commit message: New URDF model implemented

File: Simscape/URDF/urdf/SMART NS 12-1,85_ARTICOLATO.SLDASM.urdf (robot description, URDF)
Before this commit: robot SMART NS 12-1,85_ARTICOLATO.SLDASM, 7 links, 6 joints
Links:
- removed link LinkBase
- removed link LinkEE
- added link BaseLink, mass 390.843303693814; collision mesh filename=package://SMART NS 12-1,85 ARC_040128.SLDASM/meshes/BaseLin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; visual mesh filename=package://SMART NS 12-1,85 ARC_040128.SLDASM/meshes/BaseLin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
- added link Link6, mass 0.721881062345406; collision mesh filename=package://SMART NS 12-1,85 ARC_040128.SLDASM/meshes/Link6.S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; visual mesh filename=package://SMART NS 12-1,85 ARC_040128.SLDASM/meshes/Link6.S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
- link Link1: mass 45.9345542594997 -> 360.59; geometry collision mesh filename=package://SMART NS 12-1,85 ARC_040128.SLDASM/meshes/Link1.S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; visual mesh filename=package://SMART NS 12-1,85 ARC_040128.SLDASM/meshes/Link1.S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
- link Link2: mass 7.51128820326683 -> 58.964; geometry collision mesh filename=package://SMART NS 12-1,85 ARC_040128.SLDASM/meshes/Link2.S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; visual mesh filename=package://SMART NS 12-1,85 ARC_040128.SLDASM/meshes/Link2.S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
- link Link3: mass 21.7051384673217 -> 170.385336968475; geometry collision mesh filename=package://SMART NS 12-1,85 ARC_040128.SLDASM/meshes/Link3.S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; visual mesh filename=package://SMART NS 12-1,85 ARC_040128.SLDASM/meshes/Link3.S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
- link Link4: mass 5.72544149128189 -> 44.945; geometry collision mesh filename=package://SMART NS 12-1,85 ARC_040128.SLDASM/meshes/Link4.S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; visual mesh filename=package://SMART NS 12-1,85 ARC_040128.SLDASM/meshes/Link4.S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
- link Link5: mass 0.559213536738551 -> 4.38982627500557; geometry collision mesh filename=package://SMART NS 12-1,85 ARC_040128.SLDASM/meshes/Link5.S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; visual mesh filename=package://SMART NS 12-1,85 ARC_040128.SLDASM/meshes/Link5.S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
Joints:
- joint Ax1: parent LinkBase -> BaseLink
- joint Ax2: origin xyz=-0.3 0.349 -0.101 rpy=0 0 -7.8035E-05 -> xyz=-0.3 0.349 -0.101 rpy=0 0 0
- joint Ax3: origin xyz=0 0.7 0 rpy=0 0 7.8035E-05 -> xyz=0 0.7 0 rpy=0 0 0
- joint Ax5: origin xyz=-0.592 0 0 rpy=0 0 0.016135 -> xyz=-0.592 0 0 rpy=0 0 0
- joint Ax6: child LinkEE -> Link6; origin xyz=-0.092478 0 0 rpy=-1.5434 0 0 -> xyz=-0.094 0 0 rpy=0 0 0
